Commit message: Working Updates on simulation

File: src/august_description/urdf/august.xacro (robot description, xacro)
@@ -18,5 +18,5 @@
   </visual>
   <collision>
-    <origin xyz="0 0 0" rpy="0 0 0"/>
+    <origin xyz="0 0 -0.05" rpy="0 0 0"/>
     <geometry>
       <mesh filename="package://august_description/meshes/base_link.stl" scale="0.001 0.001 0.001"/>
@@ -104,27 +104,38 @@
   </collision>
 </link>
-<joint name="Revolute 47" type="continuous">
+<joint name="revolute_47" type="continuous">
   <origin xyz="-0.082471 -0.081741 0.032559" rpy="0 0 0"/>
   <parent link="base_link"/>
   <child link="a`_1"/>
   <axis xyz="-0.0 0.0 -1.0"/>
+  <limit effort="1.0" velocity="100.0"/>
+  <dynamics damping="0.01" friction="0.001"/>
 </joint>
-<joint name="Revolute 48" type="continuous">
+<joint name="revolute_48" type="continuous">
   <origin xyz="-0.084483 0.117659 0.037559" rpy="0 0 0"/>
   <parent link="base_link"/>
   <child link="b_1"/>
   <axis xyz="0.0 0.0 -1.0"/>
+  <limit effort="1.0" velocity="100.0"/>
+  <dynamics damping="0.01" friction="0.001"/>
 </joint>
-<joint name="Revolute 49" type="continuous">
+<joint name="revolute_49" type="continuous">
   <origin xyz="0.154898 0.114909 0.037559" rpy="0 0 0"/>
   <parent link="base_link"/>
   <child link="b`_1"/>
   <axis xyz="0.0 -0.0 -1.0"/>
+  <limit effort="1.0" velocity="100.0"/>
+  <dynamics damping="0.01" friction="0.001"/>
 </joint>
-<joint name="Revolute 50" type="continuous">
+<joint name="revolute_50" type="continuous">
   <origin xyz="0.154704 -0.082227 0.032573" rpy="0 0 0"/>
   <parent link="base_link"/>
   <child link="a_1"/>
   <axis xyz="-0.0 -0.0 -1.0"/>
+  <limit effort="1.0" velocity="100.0"/>
+  <dynamics damping="0.01" friction="0.001"/>
 </joint>
+<gazebo>
+  <plugin name="gazebo_ros_control" filename="libgazebo_ros_control.so"/>
+</gazebo>
 </robot>

Commit message: mmmFOoooooooooooooooooood

File: src/august_description/urdf/august.xacro (robot description, xacro)
@@ -51,5 +51,5 @@
   </inertial>
   <visual>
-    <origin xyz="0.084483 -0.117659 -0.037559" rpy="0 0 0"/>
+    <origin xyz="0.084450 -0.117659 -0.037559" rpy="0 0 0"/>
     <geometry>
       <mesh filename="package://august_description/meshes/b_1.stl" scale="0.001 0.001 0.001"/>
@@ -58,5 +58,5 @@
   </visual>
   <collision>
-    <origin xyz="0.084483 -0.117659 -0.037559" rpy="0 0 0"/>
+    <origin xyz="0.084450 -0.117659 -0.037559" rpy="0 0 0"/>
     <geometry>
       <mesh filename="package://august_description/meshes/b_1.stl" scale="0.001 0.001 0.001"/>
@@ -113,5 +113,5 @@
 </joint>
 <joint name="revolute_48" type="continuous">
-  <origin xyz="-0.084483 0.117659 0.037559" rpy="0 0 0"/>
+  <origin xyz="-0.084450 0.117659 0.037559" rpy="0 0 0"/>
   <parent link="base_link"/>
   <child link="b_1"/>
@@ -154,3 +154,22 @@
   <self_collide>false</self_collide>
 </gazebo>
+<gazebo>
+    <sensor type="imu" name="imu_sensor">
+      <always_on>true</always_on>
+      <update_rate>50</update_rate>
+      <visualize>false</visualize>
+      <topic>imu/data</topic>
+      <plugin name="imu_plugin" filename="libgazebo_ros_imu_sensor.so">
+        <ros>
+          <namespace>/august</namespace>
+          <remapping>~/out:=imu/data</remapping>
+        </ros>
+        <bodyName>base_link</bodyName>
+        <updateRate>50.0</updateRate>
+        <gaussianNoise>0.0</gaussianNoise>
+        <xyzOffset>0 0 0</xyzOffset>
+        <rpyOffset>0 0 0</rpyOffset>
+      </plugin>
+    </sensor>
+</gazebo>
 </robot>
